File: Hardware/PCB_Khess_Cash_Drawer/PCB_Khess.kicad_sch (KiCad schematic)
At the start: 13 parts, among them J1 Screw_Terminal_01x02, J2 Conn_01x02, J3 RJ11_Connector, J4 USB3_A, Q1 BUK9637-100E,118, U1 R-78B5.0-2.0

Commit message: feat: update all pcb and schematic
Parts:
- added H1, H2, H3, H4: MountingHole_Pad, MountingHole:MountingHole_2.7mm_M2.5_Pad, symbol Mechanical:MountingHole_Pad
- C1, C2: footprint (none) -> Capacitor_SMD:C_0603_1608Metric_Pad1.08x0.95mm_HandSolder
- D1: footprint (none) -> Package_TO_SOT_SMD:TO-277A
- J1: footprint (none) -> TerminalBlock_Phoenix:TerminalBlock_Phoenix_PT-1,5-2-5.0-H_1x02_P5.00mm_Horizontal
- J2: footprint (none) -> Connector_PinHeader_2.54mm:PinHeader_1x02_P2.54mm_Vertical
- J3: footprint (none) -> Connector_RJ:RJ12_Amphenol_54601-x06_Horizontal
- J4: footprint (none) -> Connector_USB:USB3_A_Molex_48406-0001_Horizontal_Stacked
- L1: footprint (none) -> Inductor_SMD:L_0603_1608Metric_Pad1.05x0.95mm_HandSolder
- Q1: footprint (none) -> Package_TO_SOT_SMD:TO-263-2
- R1, R2: footprint (none) -> Resistor_SMD:R_0603_1608Metric_Pad0.98x0.95mm_HandSolder
Connections:
- net GND: now also H1.1, H2.1, H3.1, H4.1
Other:
- note added: "Munting holes"
- moved on the sheet: D1, Q1, R1, R2
